File: PSU-Matti.kicad_pcb (KiCad board)
At the start: 2 copper layers, 98.8 x 44.5 mm, 39 parts, among them J1 Screw_Terminal_01x04, U1 LM317_3PinPackage, U2 LM337_TO220

Commit message: fix
Parts:
- >NAME (x8): footprint Connector:keystone-FASTON -> Connector:FASTON_6.35_mm
- moved >NAME 0.51 mm to (168.7, 115.8)
- moved >NAME 0.51 mm to (158.5, 115.8)
- moved >NAME 0.51 mm to (168.7, 93.9)
- moved >NAME 0.51 mm to (158.5, 93.9)
- moved >NAME 0.51 mm to (168.7, 101.5)
- moved >NAME 0.51 mm to (158.5, 101.5)
- moved >NAME 0.51 mm to (168.7, 108.1)
- moved >NAME 0.51 mm to (158.5, 108.1)
Other:
- board text added: "v01"
- board text added: "—>"
- board text added: "←"

Commit message: fix
Parts:
- removed REF** (x4): MountingHole_3mm, MountingHole:MountingHole_3mm
- added ?: 3mm, MountingHole:MountingHole_3mm, F.Cu at (169.4, 122.4)
- added ?: 3mm, MountingHole:MountingHole_3mm, F.Cu at (169.4, 87.1)
- added ?: 3mm, MountingHole:MountingHole_3mm, F.Cu at (119.7, 104.7)
- added ?: 3mm, MountingHole:MountingHole_3mm, F.Cu at (79.8, 122.4)
- added G***: LOGO, own_libraries:falshraster, B.Cu at (122.7, 106.2)
- ?: renamed from REF**; value MountingHole_3mm -> 3mm
- moved >NAME 0.32 mm to (168.7, 108.5)
- moved >NAME 0.32 mm to (158.6, 108.5)
- moved >NAME 0.13 mm to (168.7, 101.4)
- moved >NAME 0.13 mm to (158.5, 101.4)
Other:
- board text added: "Heatsink"
